File: watering_controller.brd (EAGLE design)
At the start: 51.5 x 37.9 mm, 38 parts, among them IC1 LM324D, J1 DCJ0202, T1 BC848ASMD, T2 BC848ASMD, T3 BC848ASMD

Commit message: Update smd version
Parts:
- removed BATTERY, FEUCHT, LED4, LED6, NASS, TROCKEN: (no value), led:SML0805
- removed D1: 6.8, diode:SOD80C
- removed J1: DCJ0202, con-jack:DCJ0202
- removed R10, R11, R12, R13, R14, R9: 150, resistor:M0805
- removed R15, R17, R18: 4.7k, resistor:M0805
- removed R16, R7: 10k, resistor:M0805
- removed R5: 4.3k, resistor:M0805
- removed R6: 1k, resistor:M0805
- removed R8: 220, resistor:M0805
- removed REG1: 7805DT, linear:TO252
- removed T1, T2, T3: BC848ASMD, transistor-npn:SOT23
- added 12V_J, 5V_J, PUMP_J: DCJ0202, con-jack:DCJ0202
- added C2: 0.1uF, rcl:C0805
- added Q1, Q2, Q3: BSS123, transistor-small-signal:SOT23
- C4: value 0.22uF -> 47uF; device rcl:C0805 -> rcl:A/3216-18R
- C5: value 0.1uF -> 0.1nF
- IC1: value LM324D -> NE555D; device linear:SO14 -> linear:SO08
- JP1: device jumper:JP3Q -> pinhead:1X08
- LED1: value (none) -> GREEN
- MOS1: value BSS123 -> (none); device transistor-small-signal:SOT23 -> ckr_parts:SOT23
- R1: value 100 -> 10k
- R2: value 10k -> 200
- R3: value 1.8k -> 10k
- R4: value 680 -> 1M; device resistor:M0805 -> pot:B25P
- moved R2 225.3 mm to (-52.9, -187.7), turned to 0 degrees
- moved LED1 215.6 mm to (-51.9, -182.0), turned to 0 degrees
- moved C1 202.4 mm to (-0.95, -176.1), turned to 0 degrees
- moved C3 185.1 mm to (-0.95, -163.4), turned to 0 degrees
- moved C5 164.2 mm to (-0.95, -138.0), turned to 0 degrees
- moved R3 152.6 mm to (-0.95, -125.3), turned to 0 degrees
- moved R4 144.1 mm to (-45.7, -99.9), turned to 0 degrees
- moved IC1 95.3 mm to (-50.5, -41.5)
- moved C4 88.8 mm to (-50.2, -49.8), turned to 0 degrees
- moved MOS1 78.8 mm to (-40.6, 39.4), turned to 0 degrees
- moved JP1 53.4 mm to (-24.1, 33.0), turned to 0 degrees
- moved R1 20.6 mm to (10.6, 39.1), turned to 0 degrees
Connections:
- removed net FEUCHT: JP1.3, R11.2, R12.2, R17.2, T2.2
- removed net N$10: LED1.A, R10.1
- removed net N$11: IC1.12, R3.1, R4.2
- removed net N$12: IC1.10, R4.1, R5.2
- removed net N$13: NASS.A, R9.1
- removed net N$21: FEUCHT.A, R12.1
- removed net N$22: LED4.A, R11.1
- removed net N$23: R14.1, TROCKEN.A
- removed net N$24: LED6.A, R13.1
- removed net N$5: IC1.8, T3.1
- removed net N$6: IC1.6, R6.1, R7.2
- removed net N$7: IC1.7, MOS1.1, R16.2
- removed net N$8: MOS1.2, R8.2
- removed net N$9: BATTERY.A, R8.1
- removed net NASS: JP1.1, R10.2, R18.2, R9.2, T1.2
- removed net SOIL_IN: IC1.13, IC1.2, IC1.9, JP1.2
- removed net TROCKEN: JP1.5, R13.2, R14.2, R15.2, T3.2
- new net PUMP: IC1.3, MOS1.1, R1.2
- new net PUMP_GND: C2.2, MOS1.3, PUMP_J.2, PUMP_J.3
- new net SOIL_MOIST: JP1.1
- net +5V: now also IC1.8, R4.E; no longer C1.2, C5.1, IC1.3, JP1.4, MOS1.3, REG1.2, T1.3, T2.3, T3.3
- net +9V: now also 12V_J.1, 5V_J.1, C1.1, C2.1, PUMP_J.1; no longer C4.1, J1.1, R1.2, R6.2, REG1.1
- net GND: now also 12V_J.2, 12V_J.3, 5V_J.2, 5V_J.3, C1.2, C4.-, C5.1, IC1.1, MOS1.2, R1.1; no longer BATTERY.C, C1.1, C4.2, C5.2, D1.A, FEUCHT.C, IC1.11, J1.2, J1.3, JP1.6, LED4.C, LED6.C, NASS.C, R15.1, R16.1, R17.1, R18.1, R5.1, R7.1, REG1.3, TROCKEN.C
- net N$1: now also C5.2, IC1.5; no longer R2.1, R3.2
- net N$2: now also R3.2, R4.A, R4.S; no longer IC1.1, T1.1
- net N$3: now also C4.+, IC1.6, IC1.7, R3.1; no longer D1.C, IC1.5, R1.1
- net N$4: now also LED1.A, R2.1; no longer IC1.14, T2.1
Routing:
- net SOIL_IN: track 28.4 -> 0.00 mm
- net N$6: track 24.8 -> 0.00 mm
- net N$1: track 24.4 -> 0.00 mm
- net +5V: track 22.5 -> 0.00 mm, vias 7 -> 0
- net N$3: track 18.9 -> 0.00 mm
- net N$2: track 18.2 -> 0.00 mm, vias 2 -> 0
- net N$4: track 17.1 -> 0.00 mm, vias 2 -> 0
- net N$7: track 16.8 -> 0.00 mm, vias 2 -> 0
- net N$13: track 11.0 -> 0.00 mm
- net N$23: track 11.0 -> 0.00 mm
- net N$21: track 11.0 -> 0.00 mm
- net +9V: track 9.18 -> 0.00 mm, vias 4 -> 0
- net N$12: track 8.41 -> 0.00 mm
- net N$11: track 8.36 -> 0.00 mm
- net TROCKEN: track 8.14 -> 0.00 mm
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- removed copper zone on layer 16, net +5V
- removed copper zone on layer 16, net +9V
- removed copper zone on layer 1, net GND
Other:
- board size 51.5 x 37.9 mm -> 100 x 80 mm
- board text removed: "Battery"
- board text removed: "Feucht"
- board text removed: "LED2"
- board text removed: "LED3"
- board text removed: "LED5"
- board text removed: "MOSFET Pull-Down"
- board text removed: "Nass"
- board text removed: "Trocken"
- board text removed: "Watering Indicator v2.0"
